Commit message: Add links for the infrared receivers
Approximately position and orient according to the urdf

Signed-off-by: Emerson Knapp <emerson.b.knapp@gmail.com>

File: kobuki_description/urdf/kobuki.urdf.xacro (robot description, xacro)
@@ -208,4 +208,46 @@
       </inertial>
     </link>
+    <joint name="ir_receiver_left_joint" type="fixed">
+      <origin xyz="0.1048 0.135 0.0725" rpy="${-M_PI/2} 0 0" />
+      <parent link="base_link" />
+      <child link="ir_receiver_left_link" />
+    </joint>
+    <link name="ir_receiver_left_link">
+      <inertial>
+        <mass value="0.0001" />
+        <origin xyz="0 0 0" />
+        <inertia ixx="0.0001" ixy="0.0" ixz="0.0"
+                 iyy="0.0001" iyz="0.0"
+                 izz="0.0001" />
+      </inertial>
+    </link>
+    <joint name="ir_receiver_center_joint" type="fixed">
+      <origin xyz="0.165 0.00 0.0725" rpy="0 ${M_PI/2} 0" />
+      <parent link="base_link" />
+      <child link="ir_receiver_center_link" />
+    </joint>
+    <link name="ir_receiver_center_link">
+      <inertial>
+        <mass value="0.0001" />
+        <origin xyz="0 0 0" />
+        <inertia ixx="0.0001" ixy="0.0" ixz="0.0"
+                 iyy="0.0001" iyz="0.0"
+                 izz="0.0001" />
+      </inertial>
+    </link>
+    <joint name="ir_receiver_right_joint" type="fixed">
+      <origin xyz="0.1048 -0.135 0.0725" rpy="${M_PI/2} 0 0" />
+      <parent link="base_link" />
+      <child link="ir_receiver_right_link" />
+    </joint>
+    <link name="ir_receiver_right_link">
+      <inertial>
+        <mass value="0.0001" />
+        <origin xyz="0 0 0" />
+        <inertia ixx="0.0001" ixy="0.0" ixz="0.0"
+                 iyy="0.0001" iyz="0.0"
+                 izz="0.0001" />
+      </inertial>
+    </link>
     <!-- Kobuki Gazebo simulation details -->
     <xacro:kobuki_sim/>

Commit message: Fix ir receiver transforms to put X forward and Z up
Signed-off-by: Emerson Knapp <emerson.b.knapp@gmail.com>

File: kobuki_description/urdf/kobuki.urdf.xacro (robot description, xacro)
@@ -209,5 +209,5 @@
     </link>
     <joint name="ir_receiver_left_joint" type="fixed">
-      <origin xyz="0.1048 0.135 0.0725" rpy="${-M_PI/2} 0 0" />
+      <origin xyz="0.1048 0.135 0.0725" rpy="0 0 ${M_PI/2}" />
       <parent link="base_link" />
       <child link="ir_receiver_left_link" />
@@ -223,5 +223,5 @@
     </link>
     <joint name="ir_receiver_center_joint" type="fixed">
-      <origin xyz="0.165 0.00 0.0725" rpy="0 ${M_PI/2} 0" />
+      <origin xyz="0.165 0.00 0.0725" rpy="0 0 0" />
       <parent link="base_link" />
       <child link="ir_receiver_center_link" />
@@ -237,5 +237,5 @@
     </link>
     <joint name="ir_receiver_right_joint" type="fixed">
-      <origin xyz="0.1048 -0.135 0.0725" rpy="${M_PI/2} 0 0" />
+      <origin xyz="0.1048 -0.135 0.0725" rpy="0 0 -${M_PI/2}" />
       <parent link="base_link" />
       <child link="ir_receiver_right_link" />

Commit message: Get rid of base_footprint for now, just causes rviz flickering for no gain
Signed-off-by: Emerson Knapp <emerson.b.knapp@gmail.com>

File: kobuki_description/urdf/kobuki.urdf.xacro (robot description, xacro)
@@ -11,5 +11,4 @@
   <!-- Kobuki -->
   <xacro:macro name="kobuki">
-    <link name="base_footprint"/>
     <!--
        Base link is set at the bottom of the base mould.
@@ -21,9 +20,4 @@
        to 0.352.
       -->
-    <joint name="base_joint" type="fixed">
-      <origin xyz="0 0 0.0102" rpy="0 0 0" />
-      <parent link="base_footprint"/>
-      <child link="base_link" />
-    </joint>
     <link name="base_link">
       <visual>

Commit message: Publishing bumper state as kobuki sensorstate
Signed-off-by: Emerson Knapp <emerson.b.knapp@gmail.com>

File: kobuki_description/urdf/kobuki.urdf.xacro (robot description, xacro)
@@ -50,4 +50,24 @@
       </inertial>
     </link>
+    <joint name="bumper_joint" type="fixed">
+      <parent link="base_link"/>
+      <child link="bumper_link"/>
+      <origin xyz="0 0 0" rpy="0 0 0"/>
+    </joint>
+    <link name="bumper_link">
+      <collision name="bumper">
+        <geometry>
+          <cylinder length="0.10938" radius="0.178"/>
+        </geometry>
+        <origin xyz="0.01 0.0 0.0595" rpy="0 0 0"/>
+      </collision>
+      <inertial>
+        <mass value="0.0001" />
+        <origin xyz="0 0 0" />
+        <inertia ixx="0.0001" ixy="0.0" ixz="0.0"
+                 iyy="0.0001" iyz="0.0"
+                 izz="0.0001" />
+      </inertial>
+    </link>
     <joint name="wheel_left_joint" type="continuous">
       <parent link="base_link"/>
@@ -67,4 +87,9 @@
           <cylinder length="0.0206" radius="0.035"/>
         </geometry>
+        <surface>
+          <contact>
+            <collide_without_contact>true</collide_without_contact>
+          </contact>
+        </surface>
         <origin rpy="0 0 0" xyz="0 0 0"/>
       </collision>

File: kobuki_description/urdf/kobuki_gazebo.urdf.xacro (robot description, xacro)
@@ -2,4 +2,7 @@
 <robot name="kobuki_sim" xmlns:xacro="http://ros.org/wiki/xacro">
   <xacro:macro name="kobuki_sim">
+    <gazebo reference="bumper_joint">
+      <preserveFixedJoint>true</preserveFixedJoint>
+    </gazebo>
 	  <gazebo reference="wheel_left_link">
 	    <mu1>1.0</mu1>
@@ -34,13 +37,15 @@
 	    <maxVel>1.0</maxVel>
 	  </gazebo>
-	  <gazebo reference="base_link">
+	  <gazebo reference="bumper_link">
 	    <mu1>0.3</mu1>
 	    <mu2>0.3</mu2>
 	    <sensor type="contact" name="bumpers">
+	      <plugin name="gazebo_ros_bumper" filename="libgazebo_ros_bumper.so">
+	      </plugin>
 	      <always_on>1</always_on>
-	      <update_rate>50.0</update_rate>
+	      <update_rate>10.0</update_rate>
 	      <visualize>true</visualize>
 	      <contact>
-	        <collision>base_footprint_fixed_joint_lump__base_collision</collision>
+	        <collision>bumper_link_fixed_joint_lump__bumper_collision</collision>
 	      </contact>
 	    </sensor>
@@ -145,4 +150,5 @@
           <body_name>gyro_link</body_name>
           <frame_name>gyro_link</frame_name>
+          <initial_orientation_as_reference>false</initial_orientation_as_reference>
         </plugin>
         <always_on>true</always_on>

Commit message: Add both charging pads as contactable collision models
Signed-off-by: Emerson Knapp <emerson.b.knapp@gmail.com>

File: kobuki_description/urdf/kobuki.urdf.xacro (robot description, xacro)
@@ -149,4 +149,42 @@
       </inertial>
     </link>
+    <joint name="charge_pad_left_joint" type="fixed">
+      <parent link="base_link"/>
+      <child link="charge_pad_left_link"/>
+      <origin xyz="0.1263 0.0463 0.0" rpy="0 0 0"/>
+    </joint>
+    <link name="charge_pad_left_link">
+      <inertial>
+        <mass value="0.001" />
+        <origin xyz="0 0 0" />
+        <inertia ixx="0.001" ixy="0.0" ixz="0.0"
+                 iyy="0.001" iyz="0.0"
+                 izz="0.001" />
+      </inertial>
+      <collision>
+        <geometry>
+          <box size="0.0122 0.0151 0.01"/>
+        </geometry>
+      </collision>
+    </link>
+    <joint name="charge_pad_right_joint" type="fixed">
+      <parent link="base_link"/>
+      <child link="charge_pad_right_link"/>
+      <origin xyz="0.1263 -0.0463 0.0" rpy="0 0 0"/>
+    </joint>
+    <link name="charge_pad_right_link">
+      <inertial>
+        <mass value="0.001" />
+        <origin xyz="0 0 0" />
+        <inertia ixx="0.001" ixy="0.0" ixz="0.0"
+                 iyy="0.001" iyz="0.0"
+                 izz="0.001" />
+      </inertial>
+      <collision>
+        <geometry>
+          <box size="0.0122 0.0151 0.01"/>
+        </geometry>
+      </collision>
+    </link>
     <joint name="caster_back_joint" type="fixed">
       <parent link="base_link"/>

File: kobuki_description/urdf/kobuki_gazebo.urdf.xacro (robot description, xacro)
@@ -51,4 +51,28 @@
 	    </sensor>
 	  </gazebo>
+    <gazebo reference="charge_pad_left_joint">
+      <preserveFixedJoint>true</preserveFixedJoint>
+    </gazebo>
+    <gazebo reference="charge_pad_left_link">
+      <collision>
+        <surface>
+          <contact>
+            <collide_without_contact>true</collide_without_contact>
+          </contact>
+        </surface>
+      </collision>
+    </gazebo>
+    <gazebo reference="charge_pad_right_joint">
+      <preserveFixedJoint>true</preserveFixedJoint>
+    </gazebo>
+    <gazebo reference="charge_pad_right_link">
+      <collision>
+        <surface>
+          <contact>
+            <collide_without_contact>true</collide_without_contact>
+          </contact>
+        </surface>
+      </collision>
+    </gazebo>
 	  <gazebo reference="cliff_sensor_left_link">
 	    <sensor type="ray" name="cliff_sensor_left">
